Commit message: 增加hector.urdf

File: legged_examples/hector_description/xacro/gazebo.xacro (robot description, xacro)
@@ -26,13 +26,4 @@
         <mu2>0.2</mu2>
         <material>Gazebo/DarkGrey</material>
-    </gazebo>
-     <gazebo reference="trunkcol">
-        <mu1>0.2</mu1>
-        <mu2>0.2</mu2>
-    </gazebo>
-    <gazebo reference="stick_link">
-        <mu1>0.2</mu1>
-        <mu2>0.2</mu2>
-        <material>Gazebo/White</material>
     </gazebo>
     <gazebo reference="imu_link">
@@ -80,4 +71,22 @@
         <material>Gazebo/Grey</material>
     </gazebo>
+    <gazebo reference="L_toe_f1_link">
+        <mu1>1.5</mu1>
+        <mu2>1.5</mu2>
+        <self_collide>1</self_collide>
+        <kp value="1000000.0"/>
+        <kd value="100.0"/>
+        <maxVel>1.0</maxVel>
+        <minDepth>0.00</minDepth>
+    </gazebo>
+    <gazebo reference="L_toe_f2_link">
+        <mu1>1.5</mu1>
+        <mu2>1.5</mu2>
+        <self_collide>1</self_collide>
+        <kp value="1000000.0"/>
+        <kd value="100.0"/>
+        <maxVel>1.0</maxVel>
+        <minDepth>0.00</minDepth>
+    </gazebo>
     <!--R leg -->
     <gazebo reference="R_hip">
@@ -119,3 +128,21 @@
         <material>Gazebo/Grey</material>
     </gazebo>
+    <gazebo reference="R_toe_f1_link">
+        <mu1>1.5</mu1>
+        <mu2>1.5</mu2>
+        <self_collide>1</self_collide>
+        <kp value="1000000.0"/>
+        <kd value="100.0"/>
+        <maxVel>1.0</maxVel>
+        <minDepth>0.00</minDepth>
+    </gazebo>
+    <gazebo reference="R_toe_f2_link">
+        <mu1>1.5</mu1>
+        <mu2>1.5</mu2>
+        <self_collide>1</self_collide>
+        <kp value="1000000.0"/>
+        <kd value="100.0"/>
+        <maxVel>1.0</maxVel>
+        <minDepth>0.00</minDepth>
+    </gazebo>
 </robot>

File: legged_examples/hector_description/xacro/imu.xacro (robot description, xacro)
@@ -1,4 +1,4 @@
 <?xml version="1.0"?>
-<robot xmlns:xacro="http://www.ros.org/wiki/xacro" name="imu_link">
+<robot xmlns:xacro="http://www.ros.org/wiki/xacro" name="imu">
     <xacro:macro name="IMU" params="connected_to imu_name xyz:='0 0 0' rpy:='0 0 0' ">
         <!-- Imu is fixed to the base link -->
@@ -6,8 +6,8 @@
             <origin xyz="${xyz}" rpy="${rpy}"/>
             <parent link="${connected_to}"/>
-            <child link="${imu_name}"/>
+            <child link="${imu_name}_link"/>
         </joint>
         <!-- Imu link -->
-        <link name="${imu_name}">
+        <link name="${imu_name}_link">
             <inertial>
                 <mass value="0.01"/>
@@ -25,7 +25,4 @@
             </material>
         </link>
-        <gazebo reference="${imu_name}">
-            <material>Gazebo/Orange</material>
-        </gazebo>
         <gazebo reference="${imu_name}_joint">
             <disableFixedJointLumping>true</disableFixedJointLumping>

File: legged_examples/hector_description/xacro/leg.xacro (robot description, xacro)
@@ -5,5 +5,5 @@
         <joint name="${name}_hip_joint" type="revolute">
             <xacro:insert_block name="origin"/>
-            <parent link="trunk"/>
+            <parent link="base_link"/>
             <child link="${name}_hip"/>
             <axis xyz="0 0 1"/>

File: legged_examples/hector_description/xacro/robot.xacro (robot description, xacro)
@@ -9,5 +9,4 @@
     <!-- <xacro:stairs stairs="15" xpos="0" ypos="0" zpos="0" /> -->
     <!-- Rollover Protection mode will add an additional stick on the top, use "true" or "false" to switch it. -->
-    <xacro:property name="rolloverProtection" value="false"/>
     <!-- Debug mode will hung up the robot, use "true" or "false" to switch it. -->
     <link name="base_link">
@@ -34,59 +33,5 @@
         </inertial>
     </link>
-    <xacro:IMU connected_to="base_link" imu_name="imu_link" xyz="0. 0. 0." rpy="0. 0. 0."/>
-    <xacro:if value="${(rolloverProtection == 'True')}">
-        <joint name="stick_joint" type="fixed">
-            <parent link="base_link"/>
-            <child link="stick_link"/>
-            <origin rpy="0 0 0" xyz="${0.18} 0 ${stick_length/2.0+0.08}"/>
-        </joint>
-        <link name="stick_link">
-            <visual>
-                <geometry>
-                    <cylinder length="${stick_length}" radius="${stick_radius}"/>
-                </geometry>
-                <origin rpy="0 0 0" xyz="0 0 0"/>
-                <material name="white"/>
-            </visual>
-            <collision>
-                <geometry>
-                    <cylinder length="${stick_length}" radius="${stick_radius}"/>
-                </geometry>
-                <origin rpy="0 0 0" xyz="0 0 0"/>
-            </collision>
-            <inertial>
-                <mass value="${stick_mass}"/>
-                <inertia
-                    ixx="${stick_mass / 2.0 * (stick_radius*stick_radius)}" ixy="0.0" ixz="0.0"
-                    iyy="${stick_mass / 12.0 * (3*stick_radius*stick_radius + stick_length*stick_length)}" iyz="0.0"
-                    izz="${stick_mass / 12.0 * (3*stick_radius*stick_radius + stick_length*stick_length)}"/>
-            </inertial>
-        </link>
-    </xacro:if>
-    <joint name="imu_joint" type="fixed">
-        <parent link="base_link"/>
-        <child link="imu_link"/>
-        <origin rpy="0 0 0" xyz="0 0 0"/>
-    </joint>
-    <link name="imu_link">
-        <inertial>
-            <mass value="0.001"/>
-            <origin rpy="0 0 0" xyz="0 0 0"/>
-            <inertia ixx="0.0001" ixy="0" ixz="0" iyy="0.0001" iyz="0" izz="0.0001"/>
-        </inertial>
-        <visual>
-            <origin rpy="0 0 0" xyz="0 0 0"/>
-            <geometry>
-                <box size="0.001 0.001 0.001"/>
-            </geometry>
-            <material name="red"/>
-        </visual>
-        <collision>
-            <origin rpy="0 0 0" xyz="0 0 0"/>
-            <geometry>
-                <box size=".001 .001 .001"/>
-            </geometry>
-        </collision>
-    </link>
+    <xacro:IMU connected_to="base_link" imu_name="imu" xyz="0. 0. 0." rpy="0. 0. 0."/>
     <xacro:leg name="L" mirror="1" mirror_dae="False">
         <origin rpy="0 0 0" xyz="${hip_offset_x} ${hip_offset_y} ${-hip_offset_z}"/>
