Commit message: urdf文件中接触点距离修改

File: legged_examples/hector_description/xacro/leg.xacro (robot description, xacro)
@@ -300,8 +300,8 @@
         <joint name="${name}_toe_fixed_1" type="fixed">
             <xacro:if value="${(mirror_dae == True)}">
-                <origin xyz="0.08 0.015 -0.02" rpy="0 0 0" />
+                <origin xyz="0.08 0.02 -0.02" rpy="0 0 0" />
             </xacro:if>
             <xacro:if value="${(mirror_dae == False)}">
-                <origin xyz="0.08 -0.015 -0.02" rpy="0 0 0" />
+                <origin xyz="0.08 -0.02 -0.02" rpy="0 0 0" />
             </xacro:if>
             <parent link="${name}_toe" />
@@ -328,8 +328,8 @@
         <joint name="${name}_toe_fixed_2" type="fixed">
             <xacro:if value="${(mirror_dae == True)}">
-                <origin xyz="-0.06 0.015 -0.02" rpy="0 0 0" />
+                <origin xyz="-0.06 0.02 -0.02" rpy="0 0 0" />
             </xacro:if>
             <xacro:if value="${(mirror_dae == False)}">
-                <origin xyz="-0.06 -0.015 -0.02" rpy="0 0 0" />
+                <origin xyz="-0.06 -0.02 -0.02" rpy="0 0 0" />
             </xacro:if>
             <parent link="${name}_toe" />
